File: ESP32_S3_ETH/ESP32_S3_ETH.kicad_sch (KiCad schematic)
At the start: 86 parts, among them J1 USB_C_Receptacle_USB2.0_16P, J2 USB_C_Receptacle_USB2.0_16P, J3 J1B1211CCD, Q1 L8050QLT1G, Q2 L8050QLT1G, SW1 SW_Push, SW2 SW_Push, U1 ESP32-S3-WROOM-1-N8R2, U2 CP2102N-A02-GQFN28, U3 TC1264-3.3VDB, U4 W5500, Y1 ECS-2033-250-BN-TR3

Commit message: ESP_ETH Schematic Finished, Routing Started on PCB
Parts:
- removed C1, C20: 0.1uF, Capacitor_SMD:C_0603_1608Metric, symbol Device:C_Small
- removed C21: 10uF/16V, Capacitor_Tantalum_SMD:CP_EIA-6032-28_Kemet-C, symbol Device:C_Polarized_Small_US
- removed C4: 1uF, Capacitor_SMD:C_0603_1608Metric, symbol Device:C_Small
- removed JP1: PMODE2, Jumper:SolderJumper-3_P1.3mm_Open_RoundedPad1.0x1.5mm_NumberLabels, symbol Jumper:SolderJumper_3_Open
- removed JP2: PMODE1, Jumper:SolderJumper-3_P1.3mm_Open_RoundedPad1.0x1.5mm_NumberLabels, symbol Jumper:SolderJumper_3_Open
- removed JP3: PMODE0, Jumper:SolderJumper-3_P1.3mm_Open_RoundedPad1.0x1.5mm_NumberLabels, symbol Jumper:SolderJumper_3_Open
- removed R31, R32, R33: 10K, Resistor_SMD:R_0603_1608Metric, symbol Device:R_Small_US
- removed U1: ESP32-S3-WROOM-1-N8R2, ESP32-S3-WROOM-1-N8R2:XCVR_ESP32-S3-WROOM-1-N8R2, symbol ESP32-S3-WROOM-1-N8R2:ESP32-S3-WROOM-1-N8R2
- removed U3: TC1264-3.3VDB, footprints:SOT-223_3MC_MCH-L, symbol 2024-02-08_09-36-05:TC1264-3.3VDB
- added C6: 0.1uF, Capacitor_SMD:C_0603_1608Metric, symbol Device:C_Small
- added C7: 10uF, Capacitor_SMD:C_0603_1608Metric, symbol Device:C_Small
- added H1: M3_1, MountingHole:MountingHole_3.2mm_M3_ISO14580_Pad, symbol Mechanical:MountingHole_Pad
- added H2: M3_3, MountingHole:MountingHole_3.2mm_M3_ISO14580_Pad, symbol Mechanical:MountingHole_Pad
- added H3: M3_2, MountingHole:MountingHole_3.2mm_M3_ISO14580_Pad, symbol Mechanical:MountingHole_Pad
- added H4: M3_4, MountingHole:MountingHole_3.2mm_M3_ISO14580_Pad, symbol Mechanical:MountingHole_Pad
- added IC1: TC1264-3.3VDB, KiCad:SOT230P700X180-4N, symbol TC1264-3_3VDB:TC1264-3.3VDB
- added PM0, PM1, PM2: 10K, Jumper:SolderJumper-3_P1.3mm_Open_Pad1.0x1.5mm, symbol Jumper:Jumper_3_Open
- added R34, R35, R36, R37: 0, Resistor_SMD:R_0603_1608Metric, symbol Device:R_Small_US
- added U1: ESP32-S3-WROOM-1, Espressif:ESP32-S3-WROOM-1, symbol Espressif:ESP32-S3-WROOM-1
- C2: value 10uF -> 1uF
- D3: renamed from D2; footprint Diode_SMD:D_SOD-123 -> 1N5819HW-7-F:SOD3715X145N
- D5: renamed from D4; footprint Diode_SMD:D_SOD-123 -> 1N5819HW-7-F:SOD3715X145N
- FB1: value BK0603LL121-T -> ~; footprint BK0603LL121-T:BEADC0603X33N -> fb:BEADC1608X95N
- J1, J2: footprint Connector_USB:USB_C_Receptacle_GCT_USB4085 -> Connector_USB:USB_C_Receptacle_GCT_USB4105-xx-A_16P_TopMnt_Horizontal
- R1: value 47K -> 10K; footprint Diode_SMD:D_0603_1608Metric -> Resistor_SMD:R_0603_1608Metric
- R2: value 10K -> 0; footprint Resistor_SMD:R_0603_1608Metric -> Diode_SMD:D_0603_1608Metric
- SW1: renamed from SW2; value SW_Push -> RST; footprint Button_Switch_THT:SW_PUSH_6mm -> Button_Switch_SMD:SW_SPST_B3U-1000P
- SW2: renamed from SW1; value SW_Push -> BOOT; footprint Button_Switch_THT:SW_PUSH_6mm -> Button_Switch_SMD:SW_SPST_B3U-1000P
- renumbered C8 to C1, C15 to C10, C16 to C11, C22 to C12, C17 to C13, C18 to C14, C19 to C15, C3 to C16, C24 to C17, C25 to C18, C29 to C19, C5 to C20, C26 to C21, C30 to C22, C28 to C23, C27 to C24, C7 to C25, C6 to C26, C13 to C27, C12 to C28, C10 to C3, C11 to C4, C9 to C5, C23 to C8, C14 to C9, D7 to D1, D1 to D2, D3 to D4, D5 to D6, D6 to D7, R8 to R10, R22 to R11, R26 to R12, R23 to R13, R24 to R14, R27 to R15, R25 to R16, R13 to R17, R14 to R18, R29 to R19, R30 to R20, R10 to R21, R9 to R23, R11 to R24, R12 to R25, R19 to R27, R16 to R29, R21 to R3, R15 to R30, R20 to R31, R18 to R32, R17 to R33, R28 to R4, R3 to R5, R4 to R6, R5 to R7, R6 to R8, R7 to R9, U4 to U2, U2 to U3
Connections:
- net GPIO47 is gone; now on net GPIO1: R31.1
- net CHIP_PU: now also C2.1, R1.2, U1.3 (EN); no longer R2.2
- net ESP_3V3: now also U1.2 (3V3)
- net ESP_U0_RXD0: now also U1.37 (U0TXD/GPIO43/CLK_OUT1)
- net ESP_U0_TXD0: now also U1.36 (U0RXD/GPIO44/CLK_OUT2)
- net GND: now also C6.2, C7.2, H1.1, H2.1, H3.1, H4.1, IC1.2 (GND_1), IC1.4 (GND_2), PM0.3 (B), PM1.3 (B), PM2.3 (B), U1.1 (GND), U1.40 (GND), U1.41 (GND)
- net GPIO0: now also U1.27 (GPIO0/BOOT)
- net GPIO1: now also U1.39 (GPIO1/TOUCH1/ADC1_CH0)
- net GPIO38: now also U1.31 (GPIO38/FSPIWP/SUBSPIWP)
- net INTn: now also U1.17 (GPIO9/TOUCH9/ADC1_CH8/FSPIHD/SUBSPIHD)
- net MISO: now also U1.19 (GPIO11/TOUCH11/ADC2_CH0/FSPID/FSPIIO5/SUBSPID)
- net MOSI: now also U1.18 (GPIO10/TOUCH10/ADC1_CH9/FSPICS0/FSPIIO4/SUBSPICS0)
- net PMODE0: now also PM0.2 (C)
- net PMODE1: now also PM1.2 (C)
- net PMODE2: now also PM2.2 (C)
- net RSTn: now also U1.12 (GPIO8/TOUCH8/ADC1_CH7/SUBSPICS1)
- net SCLK: now also U1.20 (GPIO12/TOUCH12/ADC2_CH1/FSPICLK/FSPIIO6/SUBSPICLK)
- net SCSn: now also U1.21 (GPIO13/TOUCH13/ADC2_CH2/FSPIQ/FSPIIO7/SUBSPIQ)
- net VCC_3V3: now also R2.2, C6.1, C7.1, IC1.3 (VOUT), PM0.1 (A), PM1.1 (A), PM2.1 (A); no longer C2.1, R1.2
- net VCC_5V: now also IC1.1 (VIN)
- net at C23.1, R12.1: now also R36.2; no longer U2.6 (RXP)
- net at C24.1, R15.1: now also R37.2; no longer U2.5 (RXN)
- net at J3.3, R13.2: now also R35.2; no longer U2.1 (TXN)
- net at J3.1, R14.2: now also R34.2; no longer U2.2 (TXP)
- net GND1 renamed CH_GND
- net GPIO19 renamed GPIO_USB-
- net GPIO_USB-: now also U1.13 (GPIO19/U1RTS/ADC2_CH8/CLK_OUT2/USB_D-)
- net GPIO20 renamed GPIO_USB+
- net GPIO_USB+: now also U1.14 (GPIO20/U1CTS/ADC2_CH9/CLK_OUT1/USB_D+)
- new net RX_N: R37.1, U2.5 (RXN)
- new net RX_P: R36.1, U2.6 (RXP)
- new net TX_N: R35.1, U2.1 (TXN)
- new net TX_P: R34.1, U2.2 (TXP)
Other:
- moved on the sheet: C16, C20, C25, C26, C27, C28, D2, D3, D4, D5, D6, D7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

Commit message: Initial commit of the routing for the ethernet PCB for review and correction.
Connections:
- net V_BUS: no longer D2.4 (K), D3.A, J1.A4 (VBUS), J1.A9 (VBUS), J1.B4 (VBUS), J1.B9 (VBUS)
- net RJ_RX_N: now reaches C19.1, J3.5, R12.2, R15.2
- net RJ_TX_P: now reaches J3.1, R14.2, R34.2
- net RJ_TX_N: now reaches J3.3, R13.2, R35.2
- net RJ_RX_P: now reaches C23.2, J3.4
- new net V_BUS_JTAG: D2.4 (K), D3.A, J1.A4 (VBUS), J1.A9 (VBUS), J1.B4 (VBUS), J1.B9 (VBUS)
Changed lines of the file:
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@@
+    (effects (font (size 1.27 1.27)) (justify left bottom))
+  )
+  (label "RJ_RX_N" (at 401.32 149.86 0) (fields_autoplaced)
     (effects (font (size 1.27 1.27)) (justify left bottom))
   )
@@
     (effects (font (size 1.27 1.27)) (justify left bottom))
   )
+  (label "RJ_RX_P" (at 401.32 144.78 0) (fields_autoplaced)
+    (effects (font (size 1.27 1.27)) (justify left bottom))
+  )
   (label "USB_D-" (at 416.56 59.69 0) (fields_autoplaced)
     (effects (font (size 1.27 1.27)) (justify left bottom))
@@
   (label "VCC_3V3" (at 400.05 160.02 180) (fields_autoplaced)
     (effects (font (size 1.27 1.27)) (justify right bottom))
+  )
+  (label "RJ_TX_P" (at 401.32 129.54 0) (fields_autoplaced)
+    (effects (font (size 1.27 1.27)) (justify left bottom))
   )
   (label "RX_N" (at 308.61 135.89 0) (fields_autoplaced)
@@
     (effects (font (size 1.27 1.27)) (justify left bottom))
   )
-  (label "V_BUS" (at 245.11 38.1 90) (fields_autoplaced)
+  (label "V_BUS_JTAG" (at 245.11 38.1 90) (fields_autoplaced)
     (effects (font (size 1.27 1.27)) (justify left bottom))
   )
@@
     (effects (font (size 1.27 1.27)) (justify right bottom))
   )
+  (label "RJ_TX_N" (at 401.32 139.7 0) (fields_autoplaced)
+    (effects (font (size 1.27 1.27)) (justify left bottom))
+  )
   (label "GPIO1" (at 139.7 44.45 0) (fields_autoplaced)

Commit message: Routing of Ethernet PCB completed, Pending further verification before finalized.
Parts:
- J3: footprint eec:WIZnet-J1B1211CCD-MFG -> Connector_RJ:RJ45_Cetus_J1B1211CCD_Horizontal
- Q1, Q2: footprint SS8050-G:TRANS_SS8050-G -> mmss8050:SOT-23_MCC
- U1: footprint Espressif:ESP32-S3-WROOM-1 -> PCM_Espressif:ESP32-S3-WROOM-1
Connections:
- net CH_GND: no longer J3.14 (MNT_2)
- net RJ_RX_N: now also C24.2, J3.6; no longer C19.1, J3.5, R12.2, R15.2
- new net: C19.1, J3.5, R12.2, R15.2
Changed lines of the file:
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@@
     (stroke (width 0) (type default))
   )
+  (wire (pts (xy 396.24 180.34) (xy 408.94 180.34))
+    (stroke (width 0) (type default))
+  )
   (wire (pts (xy 135.89 29.21) (xy 151.13 29.21))
     (stroke (width 0) (type default))
@@
     (stroke (width 0) (type default))
   )
-  (wire (pts (xy 397.51 204.47) (xy 407.67 204.47))
+  (wire (pts (xy 396.24 204.47) (xy 407.67 204.47))
     (stroke (width 0) (type default))
   )
@@
     (stroke (width 0) (type default))
   )
-  (wire (pts (xy 408.94 180.34) (xy 397.51 180.34))
-    (stroke (width 0) (type default))
-  )
   (wire (pts (xy 553.72 87.63) (xy 556.26 87.63))
     (stroke (width 0) (type default))
@@
     (stroke (width 0) (type default))
   )
-  (wire (pts (xy 388.62 154.94) (xy 408.94 154.94))
-    (stroke (width 0) (type default))
-  )
   (wire (pts (xy 215.9 196.85) (xy 215.9 199.39))
     (stroke (width 0) (type default))
@@
     (stroke (width 0) (type default))
   )
+  (wire (pts (xy 388.62 154.94) (xy 408.94 154.94))
+    (stroke (width 0) (type default))
+  )
   (wire (pts (xy 307.34 163.83) (xy 313.69 163.83))
     (stroke (width 0) (type default))
@@
     (stroke (width 0) (type default))
   )
-  (wire (pts (xy 386.08 195.58) (xy 408.94 195.58))
-    (stroke (width 0) (type default))
-  )
   (wire (pts (xy 243.84 142.24) (xy 243.84 139.7))
     (stroke (width 0) (type default))
@@
     (stroke (width 0) (type default))
   )
-  (wire (pts (xy 397.51 180.34) (xy 397.51 204.47))
+  (wire (pts (xy 396.24 180.34) (xy 396.24 204.47))
     (stroke (width 0) (type default))
   )
@@
     (effects (font (size 1.27 1.27)) (justify left bottom))
   )
-  (label "RJ_RX_N" (at 401.32 149.86 0) (fields_autoplaced)
-    (effects (font (size 1.27 1.27)) (justify left bottom))
-  )
   (label "MOSI" (at 270.51 135.89 0) (fields_autoplaced)
     (effects (font (size 1.27 1.27)) (justify left bottom))
@@
     (effects (font (size 1.27 1.27)) (justify left bottom))
   )
+  (label "RJ_RX_N" (at 402.59 154.94 0) (fields_autoplaced)
+    (effects (font (size 1.27 1.27)) (justify left bottom))
+  )
   (label "VCC_3V3" (at 99.06 128.27 90) (fields_autoplaced)
     (effects (font (size 1.27 1.27)) (justify left bottom))
@@
       (effects (font (size 1.27 1.27)) (justify left))
     )
-    (property "Footprint" "SS8050-G:TRANS_SS8050-G" (at 532.13 29.21 0)
+    (property "Footprint" "mmss8050:SOT-23_MCC" (at 532.13 29.21 0)
       (effects (font (size 1.27 1.27)) (justify bottom) hide)
     )
@@
       (effects (font (size 1.27 1.27)) (justify left))
     )
-    (property "Footprint" "SS8050-G:TRANS_SS8050-G" (at 532.13 49.53 0)
+    (property "Footprint" "mmss8050:SOT-23_MCC" (at 532.13 49.53 0)
       (effects (font (size 1.27 1.27)) (justify bottom) hide)
     )
@@
       (effects (font (size 1.27 1.27)) (justify left))
     )
-    (property "Footprint" "Espressif:ESP32-S3-WROOM-1" (at 92.71 110.49 0)
+    (property "Footprint" "PCM_Espressif:ESP32-S3-WROOM-1" (at 92.71 110.49 0)
       (effects (font (size 1.27 1.27)) hide)
     )
@@
       (effects (font (size 1.27 1.27)))
     )
-    (property "Footprint" "eec:WIZnet-J1B1211CCD-MFG" (at 406.4 116.84 0)
+    (property "Footprint" "Connector_RJ:RJ45_Cetus_J1B1211CCD_Horizontal" (at 406.4 116.84 0)
       (effects (font (size 1.27 1.27)) (justify left) hide)
     )
@@
     (pin "4")
     (pin "12")
-    (pin "14")
     (pin "10")
     (pin "1")

Commit message: Ethernet PCB finalized and ordered, hardware construction pending arrival.
Parts:
- added TP1, TP2: TestPoint, Connector_PinHeader_2.54mm:PinHeader_1x01_P2.54mm_Vertical, symbol Connector:TestPoint
- D6, D7: footprint LED_SMD:LED_SK6812_PLCC4_5.0x5.0mm_P3.2mm -> LED_SMD:LED_SK6812MINI_PLCC4_3.5x3.5mm_P1.75mm
- R2: footprint Diode_SMD:D_0603_1608Metric -> Resistor_SMD:R_0603_1608Metric
Connections:
- net VCC_3V3: now also TP2.1
- net VCC_5V: now also TP1.1
Changed lines of the file:
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@@
   (junction (at 186.69 132.08) (diameter 0) (color 0 0 0 0)
   )
+  (junction (at 264.16 40.64) (diameter 0) (color 0 0 0 0)
+  )
   (junction (at 339.09 187.96) (diameter 0) (color 0 0 0 0)
   )
@@
     (stroke (width 0) (type default))
   )
+  (wire (pts (xy 161.29 176.53) (xy 193.04 176.53))
+    (stroke (width 0) (type default))
+  )
   (wire (pts (xy 396.24 204.47) (xy 407.67 204.47))
     (stroke (width 0) (type default))
@@
     (stroke (width 0) (type default))
   )
-  (wire (pts (xy 260.35 40.64) (xy 266.7 40.64))
+  (wire (pts (xy 260.35 40.64) (xy 264.16 40.64))
     (stroke (width 0) (type default))
   )
@@
     (stroke (width 0) (type default))
   )
-  (wire (pts (xy 44.45 196.85) (xy 44.45 200.66))
-    (stroke (width 0) (type default))
-  )
   (wire (pts (xy 485.14 147.32) (xy 491.49 147.32))
     (stroke (width 0) (type default))
@@
     (stroke (width 0) (type default))
   )
+  (wire (pts (xy 264.16 40.64) (xy 266.7 40.64))
+    (stroke (width 0) (type default))
+  )
   (wire (pts (xy 495.3 139.7) (xy 516.89 139.7))
     (stroke (width 0) (type default))
@@
     (stroke (width 0) (type default))
   )
+  (wire (pts (xy 44.45 196.85) (xy 44.45 200.66))
+    (stroke (width 0) (type default))
+  )
   (wire (pts (xy 270.51 140.97) (xy 276.86 140.97))
     (stroke (width 0) (type default))
@@
     (stroke (width 0) (type default))
   )
-  (wire (pts (xy 161.29 176.53) (xy 193.04 176.53))
-    (stroke (width 0) (type default))
-  )
   (wire (pts (xy 270.51 130.81) (xy 276.86 130.81))
     (stroke (width 0) (type default))
@@
       (effects (font (size 1.27 1.27)))
     )
-    (property "Footprint" "LED_SMD:LED_SK6812_PLCC4_5.0x5.0mm_P3.2mm" (at 565.15 95.25 0)
+    (property "Footprint" "LED_SMD:LED_SK6812MINI_PLCC4_3.5x3.5mm_P1.75mm" (at 565.15 95.25 0)
       (effects (font (size 1.27 1.27)) (justify left top) hide)
     )
@@
       (effects (font (size 1.27 1.27)))
     )
-    (property "Footprint" "LED_SMD:LED_SK6812_PLCC4_5.0x5.0mm_P3.2mm" (at 523.24 95.25 0)
+    (property "Footprint" "LED_SMD:LED_SK6812MINI_PLCC4_3.5x3.5mm_P1.75mm" (at 523.24 95.25 0)
       (effects (font (size 1.27 1.27)) (justify left top) hide)
     )
@@
     )
   )
+  (symbol (lib_id "Connector:TestPoint") (at 88.9 133.35 0) (unit 1)
+    (in_bom yes) (on_board yes) (dnp no) (fields_autoplaced)
+    (property "Reference" "TP2" (at 91.44 128.778 0)
+      (effects (font (size 1.27 1.27)) (justify left))
+    )
+    (property "Value" "TestPoint" (at 91.44 131.318 0)
+      (effects (font (size 1.27 1.27)) (justify left))
+    )
+    (property "Footprint" "Connector_PinHeader_2.54mm:PinHeader_1x01_P2.54mm_Vertical" (at 93.98 133.35 0)
+      (effects (font (size 1.27 1.27)) hide)
+    )
+    (property "Datasheet" "~" (at 93.98 133.35 0)
+      (effects (font (size 1.27 1.27)) hide)
+    )
+    (pin "1")
+    (instances
+      (project "ESP32_S3_ETH"
+        (path "/25c911b0-eef6-4f9f-a9d7-5fd3483f69d6"
+          (reference "TP2") (unit 1)
+        )
+      )
+    )
+  )
   (symbol (lib_id "Device:R_Small_US") (at 339.09 129.54 90) (unit 1)
     (in_bom yes) (on_board yes) (dnp no)
@@
     )
   )
+  (symbol (lib_id "Connector:TestPoint") (at 264.16 40.64 0) (unit 1)
+    (in_bom yes) (on_board yes) (dnp no) (fields_autoplaced)
+    (property "Reference" "TP1" (at 266.7 36.068 0)
+      (effects (font (size 1.27 1.27)) (justify left))
+    )
+    (property "Value" "TestPoint" (at 266.7 38.608 0)
+      (effects (font (size 1.27 1.27)) (justify left))
+    )
+    (property "Footprint" "Connector_PinHeader_2.54mm:PinHeader_1x01_P2.54mm_Vertical" (at 269.24 40.64 0)
+      (effects (font (size 1.27 1.27)) hide)
+    )
+    (property "Datasheet" "~" (at 269.24 40.64 0)
+      (effects (font (size 1.27 1.27)) hide)
+    )
+    (pin "1")
+    (instances
+      (project "ESP32_S3_ETH"
+        (path "/25c911b0-eef6-4f9f-a9d7-5fd3483f69d6"
+          (reference "TP1") (unit 1)
+        )
+      )
+    )
+  )
   (symbol (lib_id "Device:C_Small") (at 44.45 194.31 0) (unit 1)
     (in_bom yes) (on_board yes) (dnp no) (fields_autoplaced)
@@
       (effects (font (size 1.27 1.27)))
     )
-    (property "Footprint" "Diode_SMD:D_0603_1608Metric" (at 93.98 189.23 0)
+    (property "Footprint" "Resistor_SMD:R_0603_1608Metric" (at 93.98 189.23 0)
       (effects (font (size 1.27 1.27)) hide)
     )
